File: src/hardware/quantum_monster.kicad_pcb (KiCad board)
At the start: 2 copper layers, 21 parts, among them J1 ICSP, J2 PCD8544, Q1 VS1838B, SW1 RESET, SW2 A, SW3 B, SW4 C, U1 ATmega328P-PU, Y1 32.768kHz

Commit message: Continue experimenting with hardware design.
Parts:
- added C1: 100nF, Capacitor_THT:C_Disc_D5.0mm_W2.5mm_P2.50mm, B.Cu at (187.3, 48.3)
- added C2: 100nF, Capacitor_THT:C_Disc_D5.0mm_W2.5mm_P2.50mm, B.Cu at (161.3, 53.9)
- added C3: 10uF, Capacitor_THT:C_Disc_D4.3mm_W1.9mm_P5.00mm, B.Cu at (154.3, 63.4)
- added C5: 47uF, Capacitor_THT:CP_Radial_D5.0mm_P2.00mm, F.Cu at (142.9, 38.1)
- added L1: 10uH, Inductor_THT:L_Axial_L5.3mm_D2.2mm_P7.62mm_Horizontal_Vishay_IM-1, B.Cu at (156.8, 66.0)
- added R8: 270R, Resistor_THT:R_Axial_DIN0204_L3.6mm_D1.6mm_P7.62mm_Horizontal, B.Cu at (193.7, 38.1)
- added R9: 100R, Resistor_THT:R_Axial_DIN0204_L3.6mm_D1.6mm_P7.62mm_Horizontal, F.Cu at (146.1, 38.1)
- BT1: value Battery_Cell -> CR2032
- BZ1, R3, R4, R5, R6, R7: moved to F.Cu
- C4: footprint Capacitor_THT:C_Disc_D5.0mm_W2.5mm_P5.00mm -> Capacitor_THT:C_Disc_D4.3mm_W1.9mm_P5.00mm; moved to B.Cu
- D2: footprint LED_THT:LED_D5.0mm -> LED_THT:LED_D5.0mm_IRBlack; moved to F.Cu
- Q1: footprint Package_TO_SOT_THT:TO-92_Inline_Wide -> Package_TO_SOT_THT:TO-92L_Inline_Wide; moved to F.Cu
- moved R6 146.2 mm to (174.0, 30.5), turned to 270 degrees
- moved R2 144.9 mm to (194.9, 58.4), turned to 180 degrees
- moved D2 144.1 mm to (189.9, 33.0)
- moved SW1 143.1 mm to (193.8, 67.9), turned to 180 degrees
- moved U1 133.1 mm to (179.1, 48.3), turned to 90 degrees
- moved D1 133.1 mm to (182.2, 40.6)
- moved R1 133.1 mm to (184.8, 48.3)
- moved J1 125.1 mm to (182.2, 31.8)
- moved BZ1 110.4 mm to (167.6, 32.2), turned to 270 degrees
- moved C4 102.5 mm to (151.1, 63.4), turned to 90 degrees
- moved SW4 98.9 mm to (187.3, 61.0)
- moved SW3 98.8 mm to (187.3, 51.1)
- moved SW2 98.7 mm to (187.3, 41.2)
- moved J2 98.3 mm to (162.6, 53.3)
- moved BT1 95.4 mm to (172.7, 62.2), turned to 90 degrees
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Connections:
- net LCDCLK renamed DISPLAY_CLOCK
- net LCDMOSI renamed DISPLAY_MOSI
- BZ1 pad 2: Net-(BZ1-Pad2) -> GND
- D2 pad 1: Net-(D2-Pad1) -> GND
- J2 pad 1: LCDRESET -> DISPLAY_RESET
- J2 pad 6: LCDDATACOMMAND -> DISPLAY_DATA_COMMAND
- Q1 pad 2: Net-(Q1-Pad2) -> GND
- Q1 pad 3: Net-(Q1-Pad3) -> LINK_RECEIVER_DATA
- R7 pad 2: Net-(R7-Pad2) -> SPEAKER
- SW2 pad 1: Net-(SW2-Pad1) -> GND
- SW2 pad 2: Net-(SW2-Pad2) -> A_BUTTON
- SW3 pad 1: Net-(SW3-Pad1) -> GND
- SW3 pad 2: Net-(SW3-Pad2) -> B_BUTTON
- SW4 pad 1: Net-(SW4-Pad1) -> GND
- SW4 pad 2: Net-(SW4-Pad2) -> C_BUTTON
- U1 pad 12: Net-(U1-Pad12) -> SPEAKER
- U1 pad 15: Net-(U1-Pad15) -> LINK_TRANSMITTER
- U1 pad 20: VCC -> FILTERED_VCC
- U1 pad 23: Net-(U1-Pad23) -> A_BUTTON
- U1 pad 24: Net-(U1-Pad24) -> B_BUTTON
- U1 pad 25: Net-(U1-Pad25) -> C_BUTTON
- U1 pad 27: Net-(U1-Pad27) -> LINK_RECEIVER_DATA
- U1 pad 28: Net-(U1-Pad28) -> LINK_RECEIVER_POWER
- U1 pad 4: Net-(U1-Pad4) -> DISPLAY_RESET
- U1 pad 5: Net-(U1-Pad5) -> DISPLAY_DATA_COMMAND
- U1 pad 7: VCC -> FILTERED_VCC
Routing:
- net FILTERED_VCC: track 0.00 -> 13.1 mm
- net GND: track 0.00 -> 9.92 mm
- net VCC: track 0.00 -> 3.67 mm
