File: src/hardware/pcb/quantum_monster.sch (KiCad schematic (older format))
At the start: 28 parts, among them J1 ICSP, J2 PCD8544, Q1 VS1838B, SW1 RESET, SW2 A, SW3 B, SW4 C, U1 ATmega328P-PU, Y1 32.768kHz

Commit message: Continue PCB design.
Connections:
- net A_BUTTON: no longer U1.23 (PC0)
- net B_BUTTON: no longer U1.24 (PC1)
- net DISPLAY_DATA_COMMAND: now also U1.11 (PD5); no longer U1.5 (PD3)
- net DISPLAY_RESET: now also U1.24 (PC1); no longer U1.4 (PD2)
- net GND: now also R2.1; no longer SW1.2 (B)
- net RESET: now also SW1.2 (B); no longer R2.2
- net at SW1.1 (A): now also R2.2; no longer R2.1
- no-connect marks 5 -> 4
Other:
- moved on the sheet: R2, SW1
Changed lines of the file:
@@
 	1    0    0    -1
 $EndComp
-Text GLabel 7300 4050 2    50   Output ~ 0
+Text GLabel 7300 4250 2    50   Output ~ 0
 DISPLAY_DATA_COMMAND
-Text GLabel 7300 3950 2    50   Output ~ 0
-DISPLAY_RESET
 Text GLabel 7300 4350 2    50   Output ~ 0
 SPEAKER
-Text GLabel 7300 2950 2    50   Input ~ 0
+Text GLabel 8150 2600 2    50   Input ~ 0
 A_BUTTON
-Text GLabel 7300 3050 2    50   Input ~ 0
+Text GLabel 8350 2800 2    50   Input ~ 0
 B_BUTTON
 Text GLabel 7300 3150 2    50   Input ~ 0
@@
 Wire Wire Line
 	1000 1250 950  1250
-Connection ~ 1000 1950
 Wire Wire Line
 	1400 1950 1000 1950
@@
 Connection ~ 1400 1250
 $Comp
-L Switch:SW_SPST SW1
-U 1 1 61D00CAA
-P 1000 1750
-F 0 "SW1" V 954 1848 50  0000 L CNN
-F 1 "RESET" V 1045 1848 50  0000 L CNN
-F 2 "Button_Switch_THT:SW_TH_Tactile_Omron_B3F-10xx" H 1000 1750 50  0001 C CNN
-F 3 "~" H 1000 1750 50  0001 C CNN
-	1    1000 1750
-	0    1    1    0
-$EndComp
-$Comp
-L Device:R R2
-U 1 1 61CFFBE6
-P 1000 1400
-F 0 "R2" H 930 1354 50  0000 R CNN
-F 1 "330R" H 930 1445 50  0000 R CNN
-F 2 "Resistor_THT:R_Axial_DIN0204_L3.6mm_D1.6mm_P7.62mm_Horizontal" V 930 1400 50  0001 C CNN
-F 3 "~" H 1000 1400 50  0001 C CNN
-	1    1000 1400
-	-1   0    0    1
-$EndComp
-$Comp
 L Device:C C1
 U 1 1 61CFF275
@@
 Text Notes 1950 600  0    50   ~ 0
 POWER
-NoConn ~ 7300 3750
+Text GLabel 7300 3050 2    50   Output ~ 0
+DISPLAY_RESET
+$Comp
+L Device:R R2
+U 1 1 61CFFBE6
+P 1000 1800
+F 0 "R2" H 930 1754 50  0000 R CNN
+F 1 "330R" H 930 1845 50  0000 R CNN
+F 2 "Resistor_THT:R_Axial_DIN0204_L3.6mm_D1.6mm_P7.62mm_Horizontal" V 930 1800 50  0001 C CNN
+F 3 "~" H 1000 1800 50  0001 C CNN
+	1    1000 1800
+	-1   0    0    1
+$EndComp
+Connection ~ 1000 1950
+$Comp
+L Switch:SW_SPST SW1
+U 1 1 61D00CAA
+P 1000 1450
+F 0 "SW1" V 954 1548 50  0000 L CNN
+F 1 "RESET" V 1045 1548 50  0000 L CNN
+F 2 "Button_Switch_THT:SW_TH_Tactile_Omron_B3F-10xx" H 1000 1450 50  0001 C CNN
+F 3 "~" H 1000 1450 50  0001 C CNN
+	1    1000 1450
+	0    1    -1   0
+$EndComp
 $EndSCHEMATC

Commit message: Reduce PCB size.
Parts:
- Y1: footprint Crystal:Crystal_C38-LF_D3.0mm_L8.0mm_Horizontal -> Crystal:Crystal_C38-LF_D3.0mm_L8.0mm_Vertical
Changed lines of the file:
@@
 F 0 "Y1" H 3250 4568 50  0000 C CNN
 F 1 "32.768kHz" H 3250 4477 50  0000 C CNN
-F 2 "Crystal:Crystal_C38-LF_D3.0mm_L8.0mm_Horizontal" H 3250 4300 50  0001 C CNN
+F 2 "Crystal:Crystal_C38-LF_D3.0mm_L8.0mm_Vertical" H 3250 4300 50  0001 C CNN
 F 3 "~" H 3250 4300 50  0001 C CNN
 	1    3250 4300
