File: src/hardware/pcb/quantum_monster.kicad_sch (KiCad schematic)
At the start: 28 parts, among them J1 ICSP, J2 PCD8544, Q1 VS1838B, SW1 RESET, SW2 A, SW3 B, SW4 C, U1 ATmega328P-PU, Y1 32.768kHz

Commit message: Initial production prototype of PCB.
Parts:
- C5: symbol Device:CP -> Device:C_Polarized
- U1: symbol MCU_Microchip_ATmega:ATmega328P-PU -> MCU_Microchip_ATmega:ATmega328P-P
Connections:
- net A_BUTTON: now also SW2.1 (A), U1.2 (PD0); no longer SW2.2 (B)
- net B_BUTTON: now also U1.11 (PD5)
- net C_BUTTON: now also U1.13 (PD7); no longer U1.25 (PC2)
- net GND: now also SW2.2 (B); no longer SW2.1 (A)
- net SPEAKER: now also U1.15 (PB1); no longer U1.12 (PD6)
- net DISPLAY_RES: now reaches U1.23 (PC0)
- net DISPLAY_RES: now also J2.1 (Pin_1)
- net INFRARED_RECEIVER_POWER: now reaches U1.4 (PD2)
- net INFRARED_RECEIVER_POWER: now also R9.2
- net DISPLAY_CLOCK renamed DISPLAY_SCLK
- net DISPLAY_DATA_COMMAND renamed DISPLAY_DC
- net DISPLAY_DC: now also U1.24 (PC1); no longer U1.11 (PD5)
- net DISPLAY_MOSI renamed DISPLAY_SDIN
- removed net DISPLAY_RESET: J2.1 (Pin_1), U1.24 (PC1)
- net LINK_RECEIVER_DATA: no longer names the net of U1.27 (PC4)
- net LINK_RECEIVER_DATA: no longer Q1.3 (B)
- net LINK_RECEIVER_POWER renamed INFRARED_RECEIVER_OUT
- net INFRARED_RECEIVER_OUT: now also Q1.3 (B); no longer R9.2
- net LINK_TRANSMITTER renamed INFRARED_TRANSMITTER
- net INFRARED_TRANSMITTER: now also U1.12 (PD6); no longer U1.15 (PB1)
- no-connect marks 4 -> 8
Other:
- moved on the sheet: BT1, C2, C3, C5, D2, J1, L1, Q1, R3, R4, R5, R6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
